File: Hardware/Room 2/Room2/Room2.kicad_sch (KiCad schematic)
At the start: 6 parts, among them Q1 BC557, SW1 SW_Push, SW2 SW_Push

Commit message: Update room 2 schematic.
Parts:
- added R2, R3, R4: ?, symbol Device:R
Connections:
- new net: D1.4 (BA), R4.1
- new net: Q1.1 (C), R2.2, R3.2, R4.2
- new net: D1.2 (RA), R2.1
- new net: D1.3 (GA), R3.1
Other:
- moved on the sheet: D1
