File: Hardware/Control panel (LCD and buttons)/ControlPanel/ControlPanel.kicad_sch (KiCad schematic)
At the start: 9 parts, among them J1 LCD

Commit message: updated
Parts:
- gave numbers to parts that had none: 4
Connections:
- net at UP.1: now also A?.10 (D7); no longer A?.12 (D9)
- net at OK.1: now also A?.14 (D11); no longer A?.13 (D10)
- net at BACK.1: now also A?.15 (D12); no longer A?.10 (D7)
Changed lines of the file:
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@@
 	(wire
 		(pts
-			(xy 158.75 154.94) (xy 40.64 154.94)
+			(xy 45.72 132.08) (xy 46.99 132.08)
 		)
 		(stroke
@@
 	(wire
 		(pts
+			(xy 44.45 147.32) (xy 44.45 129.54)
+		)
+		(stroke
+			(width 0)
+			(type default)
+		)
+	)
+	(wire
+		(pts
 			(xy 41.91 40.64) (xy 52.07 40.64)
 		)
@@
 	(wire
 		(pts
-			(xy 40.64 154.94) (xy 40.64 116.84)
-		)
-		(stroke
-			(width 0)
-			(type default)
-		)
-	)
-	(wire
-		(pts
 			(xy 83.82 40.64) (xy 83.82 142.24)
 		)
@@
 	(wire
 		(pts
+			(xy 44.45 129.54) (xy 46.99 129.54)
+		)
+		(stroke
+			(width 0)
+			(type default)
+		)
+	)
+	(wire
+		(pts
 			(xy 41.91 119.38) (xy 46.99 119.38)
 		)
@@
 	(wire
 		(pts
+			(xy 43.18 149.86) (xy 43.18 116.84)
+		)
+		(stroke
+			(width 0)
+			(type default)
+		)
+	)
+	(wire
+		(pts
 			(xy 168.91 38.1) (xy 168.91 24.13)
 		)
@@
 	(wire
 		(pts
+			(xy 158.75 154.94) (xy 45.72 154.94)
+		)
+		(stroke
+			(width 0)
+			(type default)
+		)
+	)
+	(wire
+		(pts
 			(xy 152.4 34.29) (xy 152.4 24.13)
 		)
@@
 	(wire
 		(pts
+			(xy 43.18 116.84) (xy 46.99 116.84)
+		)
+		(stroke
+			(width 0)
+			(type default)
+		)
+	)
+	(wire
+		(pts
 			(xy 152.4 24.13) (xy 135.89 24.13)
 		)
@@
 	(wire
 		(pts
-			(xy 44.45 147.32) (xy 44.45 124.46)
-		)
-		(stroke
-			(width 0)
-			(type default)
-		)
-	)
-	(wire
-		(pts
 			(xy 52.07 40.64) (xy 60.96 40.64)
 		)
@@
 	(wire
 		(pts
-			(xy 44.45 124.46) (xy 46.99 124.46)
-		)
-		(stroke
-			(width 0)
-			(type default)
-		)
-	)
-	(wire
-		(pts
 			(xy 78.74 73.66) (xy 78.74 129.54)
 		)
@@
 	(wire
 		(pts
-			(xy 40.64 116.84) (xy 46.99 116.84)
+			(xy 45.72 154.94) (xy 45.72 132.08)
 		)
 		(stroke
@@
 	(wire
 		(pts
-			(xy 43.18 149.86) (xy 43.18 121.92)
-		)
-		(stroke
-			(width 0)
-			(type default)
-		)
-	)
-	(wire
-		(pts
 			(xy 139.7 149.86) (xy 43.18 149.86)
 		)
@@
 		(pts
 			(xy 125.73 38.1) (xy 113.03 38.1)
-		)
-		(stroke
-			(width 0)
-			(type default)
-		)
-	)
-	(wire
-		(pts
-			(xy 43.18 121.92) (xy 46.99 121.92)
 		)
 		(stroke
@@
 		(dnp no)
 		(fields_autoplaced yes)
-		(property "Reference" "SW?"
+		(property "Reference" "UP"
 			(at 147.32 26.67 0)
 			(effects
@@
 			(project "test"
 				(path "/0e23c15d-d18e-4bc4-b815-b9b273b3f9c0"
-					(reference "SW?")
+					(reference "UP")
 					(unit 1)
 				)
@@
 		(dnp no)
 		(fields_autoplaced yes)
-		(property "Reference" "RV?"
+		(property "Reference" "RV1"
 			(at 177.8 54.6099 0)
 			(effects
@@
 			(project "test"
 				(path "/0e23c15d-d18e-4bc4-b815-b9b273b3f9c0"
-					(reference "RV?")
+					(reference "RV1")
 					(unit 1)
 				)
@@
 		(dnp no)
 		(fields_autoplaced yes)
-		(property "Reference" "SW?"
+		(property "Reference" "BACK"
 			(at 163.83 30.48 0)
 			(effects
@@
 			(project "test"
 				(path "/0e23c15d-d18e-4bc4-b815-b9b273b3f9c0"
-					(reference "SW?")
+					(reference "BACK")
 					(unit 1)
 				)
@@
 	)
 	(symbol
+		(lib_name "SW_Push_3")
 		(lib_id "Switch:SW_Push")
 		(at 147.32 45.72 0)
@@
 		(dnp no)
 		(fields_autoplaced yes)
-		(property "Reference" "SW?"
+		(property "Reference" "DOWN"
 			(at 147.32 38.1 0)
 			(effects
@@
 			(project "test"
 				(path "/0e23c15d-d18e-4bc4-b815-b9b273b3f9c0"
-					(reference "SW?")
-					(unit 1)
-				)
+					(reference "DOWN")
+					(unit 1)
+				)
