File: Hardware/Schematic_and_PCB/Arduino Main PCB/Arduino Main PCB.kicad_sch (KiCad schematic)
At the start: 82 parts, among them J1 PIR_sensor, J10 LED_Room_2, J11 LED_Room_3, J12 LED_DOOR, J13 Buttons_Room_2, J14 Barrel_Jack, J15 Power switch, J2 Control_Panel, J3 Buttons_Room_3, J4 Buttons_Room_1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

Commit message: Some value specifier rewrite.
Parts:
- C2: value 4.7mu -> 4.7uF
Changed lines of the file:
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@@
 			)
 		)
-		(property "Value" "4.7mu"
+		(property "Value" "4.7uF"
 			(at 177.8 91.8209 0)
 			(effects
